Commit message: Refactor CouligligBot initialization and comment out unused configurations in launch and URDF files

File: src/couliglig/resource/couliglig_bot.urdf (robot description, URDF)
Before this commit: robot couliglig_bot, 9 links, 8 joints
Links:
- removed link base_link
- removed link inertial unit
- removed link lidar
- removed link solid
- removed link solid(1)
- removed link solid(2)
- removed link solid_0
- removed link solid_1
- removed link solid_3
Joints:
- removed joint base_link_solid_joint
- removed joint hingejoint
- removed joint hingejoint_2
- removed joint left_motor
- removed joint right_motor
- removed joint solid_inertial unit_joint
- removed joint solid_lidar_joint
- removed joint solid_solid(2)_joint

Commit message: Add robot state publisher and update LiDAR transform in URDF

File: src/couliglig/resource/couliglig_bot.urdf (robot description, URDF)
Before this commit: robot couliglig_bot, 0 links, 0 joints
Links:
- added link LDS-01
- added link base_link
Joints:
- added joint base_to_lidar: type fixed, parent base_link, child LDS-01, origin xyz=-0.15 -0.0086 0.1696 rpy=0 0 3.141593

Commit message: Fix LiDAR transform parameters and update EKF configuration for improved localization

File: src/couliglig/resource/couliglig_bot.urdf (robot description, URDF)
Before this commit: robot couliglig_bot, 2 links, 1 joints
Links:
- removed link LDS-01
- removed link base_link
Joints:
- removed joint base_to_lidar
